File: kicadProject/nc1.sch (KiCad schematic (older format))
At the start: 72 parts, among them J1 Conn_01x02, J2 Conn_01x03, Q1 AOB414, Q2 AOB414, Q4 BD911, U1 NCP1034, U2 NE5534, U3 NE5534

Commit message: fixes
Parts:
- U2, U3: value NE5534 -> NE5230
Changed lines of the file:
@@
 P 2000 4850
 F 0 "U2" H 1650 4650 50  0000 L CNN
-F 1 "NE5534" H 1600 4550 50  0000 L CNN
+F 1 "NE5230" H 1600 4550 50  0000 L CNN
 F 2 "Package_SO:SOIC-8_3.9x4.9mm_P1.27mm" H 2050 4900 50  0001 C CNN
 F 3 "http://www.ti.com/lit/ds/symlink/ne5534.pdf" H 2050 5000 50  0001 C CNN
@@
 P 4500 5450
 F 0 "U3" H 4000 5350 50  0000 L CNN
-F 1 "NE5534" H 3950 5250 50  0000 L CNN
+F 1 "NE5230" H 3950 5250 50  0000 L CNN
 F 2 "Package_SO:SOIC-8_3.9x4.9mm_P1.27mm" H 4550 5500 50  0001 C CNN
 F 3 "http://www.ti.com/lit/ds/symlink/ne5534.pdf" H 4550 5600 50  0001 C CNN

Commit message: more compensatioon
Parts:
- added C18: 470n, Capacitor_SMD:C_1206_3216Metric_Pad1.33x1.80mm_HandSolder, symbol Device:C
- added R25: 4.7k, Resistor_SMD:R_1206_3216Metric_Pad1.30x1.75mm_HandSolder, symbol Device:R
- U2, U3: value NE5230 -> NE5534
Connections:
- net GND: now also R25.1
- net at D10.2 (A), D11.2 (A), R21.1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: now also C18.1
- new net: C18.2, R25.2
Changed lines of the file:
@@
 P 2000 4850
 F 0 "U2" H 1650 4650 50  0000 L CNN
-F 1 "NE5230" H 1600 4550 50  0000 L CNN
+F 1 "NE5534" H 1600 4550 50  0000 L CNN
 F 2 "Package_SO:SOIC-8_3.9x4.9mm_P1.27mm" H 2050 4900 50  0001 C CNN
 F 3 "http://www.ti.com/lit/ds/symlink/ne5534.pdf" H 2050 5000 50  0001 C CNN
@@
 P 4500 5450
 F 0 "U3" H 4000 5350 50  0000 L CNN
-F 1 "NE5230" H 3950 5250 50  0000 L CNN
+F 1 "NE5534" H 3950 5250 50  0000 L CNN
 F 2 "Package_SO:SOIC-8_3.9x4.9mm_P1.27mm" H 4550 5500 50  0001 C CNN
 F 3 "http://www.ti.com/lit/ds/symlink/ne5534.pdf" H 4550 5600 50  0001 C CNN
@@
 Wire Wire Line
 	4100 6200 4100 5550
+$Comp
+L Device:C C18
+U 1 1 6080FE58
+P 4800 6550
+F 0 "C18" V 5050 6600 50  0000 C CNN
+F 1 "470n" V 4950 6600 50  0000 C CNN
+F 2 "Capacitor_SMD:C_1206_3216Metric_Pad1.33x1.80mm_HandSolder" H 4838 6400 50  0001 C CNN
+F 3 "~" H 4800 6550 50  0001 C CNN
+	1    4800 6550
+	1    0    0    -1
+$EndComp
+$Comp
+L Device:R R25
+U 1 1 60811B0D
+P 4800 6850
+F 0 "R25" V 4593 6850 50  0000 C CNN
+F 1 "4.7k" V 4684 6850 50  0000 C CNN
+F 2 "Resistor_SMD:R_1206_3216Metric_Pad1.30x1.75mm_HandSolder" V 4730 6850 50  0001 C CNN
+F 3 "~" H 4800 6850 50  0001 C CNN
+	1    4800 6850
+	-1   0    0    1
+$EndComp
+$Comp
+L power:GND #PWR0130
+U 1 1 60812927
+P 4800 7000
+F 0 "#PWR0130" H 4800 6750 50  0001 C CNN
+F 1 "GND" H 4805 6827 50  0000 C CNN
+F 2 "TestPoint:TestPoint_THTPad_3.0x3.0mm_Drill1.5mm" H 4805 6736 50  0001 C CNN
+F 3 "" H 4800 7000 50  0001 C CNN
+	1    4800 7000
+	1    0    0    -1
+$EndComp
+Connection ~ 4800 6400
 $EndSCHEMATC

Commit message: stability fixes
Parts:
- removed D9: 5V, Diode_SMD:D_MELF, symbol Device:D_Zener
- removed TP1: CurrAmp, Connector_Wire:SolderWirePad_1x01_Drill2mm, symbol Connector:TestPoint
- removed TP10: GND mpp, Connector_Wire:SolderWirePad_1x01_Drill2mm, symbol Connector:TestPoint
- removed TP11: FB mpp, Connector_Wire:SolderWirePad_1x01_Drill2mm, symbol Connector:TestPoint
- removed TP12: Vout mpp, Connector_Wire:SolderWirePad_1x01_Drill2mm, symbol Connector:TestPoint
- removed TP13: GND reg, Connector_Wire:SolderWirePad_1x01_Drill2mm, symbol Connector:TestPoint
- removed TP2: 15V, Connector_Wire:SolderWirePad_1x01_Drill2mm, symbol Connector:TestPoint
- removed TP4: 15V mpp, Connector_Wire:SolderWirePad_1x01_Drill2mm, symbol Connector:TestPoint
- removed TP8: Vin mpp, Connector_Wire:SolderWirePad_1x01_Drill2mm, symbol Connector:TestPoint
- removed TP9: 100V reg, Connector_Wire:SolderWirePad_1x01_Drill2mm, symbol Connector:TestPoint
- added C19: 100u, Capacitor_THT:CP_Radial_D5.0mm_P2.50mm, symbol Device:C
- added C20: C, Capacitor_SMD:C_1206_3216Metric_Pad1.33x1.80mm_HandSolder, symbol Device:C
- added C21: ----, Capacitor_SMD:C_1206_3216Metric_Pad1.33x1.80mm_HandSolder, symbol Device:C
- added C22: 100n, Capacitor_SMD:C_1206_3216Metric_Pad1.33x1.80mm_HandSolder, symbol Device:C
- added D9: 100v, Diode_SMD:D_SMC_Handsoldering, symbol Device:D
- added J3: Conn_01x06_Female, Connector_PinHeader_2.54mm:PinHeader_1x06_P2.54mm_Vertical, symbol Connector:Conn_01x06_Female
- added R26: -, Resistor_SMD:R_1206_3216Metric_Pad1.30x1.75mm_HandSolder, symbol Device:R
- C18: value 470n -> 100u; footprint Capacitor_SMD:C_1206_3216Metric_Pad1.33x1.80mm_HandSolder -> Capacitor_THT:CP_Radial_D5.0mm_P2.50mm
- C3: value 100n -> 22u
- C5: value 10n -> 400n
- R11: value 10k -> 4.7k
- R18: value 470 -> 220
- R25: value 4.7k -> 47k
Connections:
- net +15V: now also C18.2, J3.2 (Pin_2)
- net CurrLimGND: now also C21.2
- net FB: now also J3.5 (Pin_5)
- net GND: now also C18.1, C19.2, C21.1, J3.4 (Pin_4); no longer D6.2 (A), R25.1
- net Vin: now also J3.6 (Pin_6)
- net at C4.1, L1.1, Q1.3 (S)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: no longer D6.1 (K)
- net at --2.1, D2.1 (K), R2.2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: now also C20.1
- net Vout: now reaches C1.1, C11.1, C12.1, C9.1, D3.1 (K), L1.2, R3.1
- net Vout: now also D6.2 (A), R25.1, D9.2 (A), J3.3 (Pin_3); no longer J2.1 (Pin_1)
- net at R17.2, R9.2, U2.2 (-): now also C22.1, R26.1
- net Csense: now reaches D7.2 (A), D8.2 (A), R17.1, U2.6
- net Csense: now also C22.2, J3.1 (Pin_1)
- net at R6.1, R9.1: now also R26.2
- net at R24.2, U3.3 (+): now also C19.1
- net at D10.2 (A), D11.2 (A), R21.1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: no longer C18.1
- net at R25.2: now also C20.2; no longer C18.2
- new net: D6.1 (K), D9.1 (K), J2.1 (Pin_1)
Other:
- moved on the sheet: J2
