File: kicadProject/nc1.kicad_pcb (KiCad board)
At the start: 2 copper layers, 68 parts, among them J1 Conn_01x02, J2 Conn_01x03, Q1 2N7002, Q2 2N7002, Q4 BD911, U1 NCP1034, U2 NE5534, U3 NE5534

Commit message: more compensatioon
Parts:
- added C18: 470n, Capacitor_SMD:C_1206_3216Metric_Pad1.33x1.80mm_HandSolder, F.Cu at (71.7, 44.7)
- added R25: 4.7k, Resistor_SMD:R_1206_3216Metric_Pad1.30x1.75mm_HandSolder, F.Cu at (66.6, 43.6)
- C1: value C -> 100n; footprint Capacitor_THT:CP_Radial_D14.0mm_P5.00mm -> Capacitor_THT:CP_Radial_D18.0mm_P7.50mm
- C10: value C -> 100u
- C11, C8: value C -> 10u
- C12, C13: value C -> 100n
- C14: value C -> 100n; footprint Capacitor_THT:CP_Radial_D14.0mm_P5.00mm -> Capacitor_THT:CP_Radial_D16.0mm_P7.50mm
- C4: value 100nF -> 100nF 200V
- C5: value C -> 10n
- C9: value C -> 20u
- D1: value bav21 -> BAV21
- D11: value LED -> YELLOW
- D3: value LED -> GREEN
- D4: value D_Zener -> 15V
- D5: value D_Zener -> 5V
- D8: value LED -> RED
- L1: value INDUCTOR -> 100uH
- Q1, Q2: value 2N7002 -> AOB414
- R10, R8: value R -> 10k
- R11: value 4.7k -> 10k
- R13, R16: value R -> 0.27
- R15: value 5k -> 10k
- R18, R22: value 47k -> 470
- R19: value 10k -> 100k
- R2: value R_POT -> 20k
- R23: value 10k -> 0
- R24: value R_POT -> 100k
- R3: value R -> 47k
- R4: value 100k -> 220k
- R5: value 5k -> 12k
- R9: value R_POT -> 10k
- moved R21 0.56 mm to (71.7, 42.4)
- moved R5 0.39 mm to (67.2, 48.2), turned to 0 degrees
Connections:
- R2 pad 3: (no net) -> Net-(R2-Pad3)
- TP4 pad 1: Net-(D7-Pad2) -> 15V
- U2 pad 1: (no net) -> Net-(U2-Pad1)
- U2 pad 8: (no net) -> Net-(U2-Pad8)
- U3 pad 1: (no net) -> Net-(U3-Pad1)
- U3 pad 8: (no net) -> Net-(U3-Pad8)
Routing:
- net Net-(C18-Pad2): track 0.00 -> 2.49 mm
- net Net-(D9-Pad1): track 13.9 -> 16.4 mm
- net Net-(C18-Pad1): track 74.3 -> 76.7 mm
- net Net-(R4-Pad1): track 7.33 -> 8.67 mm

Commit message: stability fixes
Parts:
- removed TP10: GND mpp, Connector_Wire:SolderWire-0.1sqmm_1x01_D0.4mm_OD1mm
- removed TP11: FB mpp, Connector_Wire:SolderWire-0.1sqmm_1x01_D0.4mm_OD1mm
- removed TP12: Vout mpp, Connector_Wire:SolderWire-0.1sqmm_1x01_D0.4mm_OD1mm
- removed TP4 (x2): 15V mpp, Connector_Wire:SolderWire-0.1sqmm_1x01_D0.4mm_OD1mm
- removed TP8: Vin mpp, Connector_Wire:SolderWire-0.1sqmm_1x01_D0.4mm_OD1mm
- added C19: 100u, Capacitor_THT:CP_Radial_D5.0mm_P2.50mm, F.Cu at (77.7, 51.8)
- added C20: C, Capacitor_SMD:C_1206_3216Metric_Pad1.33x1.80mm_HandSolder, F.Cu at (53.7, 46.3)
- added C21: 470n, Capacitor_SMD:C_1206_3216Metric_Pad1.33x1.80mm_HandSolder, F.Cu at (21.6, 61.4)
- added C22: 100n, Capacitor_SMD:C_1206_3216Metric_Pad1.33x1.80mm_HandSolder, F.Cu at (27.7, 43.2)
- added D6: 100v, Diode_SMD:D_SMC_Handsoldering, F.Cu at (26.8, 82.0)
- added D9: 100v, Diode_SMD:D_SMC_Handsoldering, F.Cu at (26.7, 87.1)
- added J3: Conn_01x06_Female, Connector_PinHeader_2.54mm:PinHeader_1x06_P2.54mm_Vertical, F.Cu at (30.3, 40.0)
- added R26: -, Resistor_SMD:R_1206_3216Metric_Pad1.30x1.75mm_HandSolder, F.Cu at (27.2, 51.2)
- C18: value 470n -> 100u; footprint Capacitor_SMD:C_1206_3216Metric_Pad1.33x1.80mm_HandSolder -> Capacitor_THT:CP_Radial_D5.0mm_P2.50mm
- C3: value 100n -> 22u
- C5: value 10n -> 400n
- R11: value 10k -> 4.7k
- R18: value 470 -> 220
- R25: value 4.7k -> 47k
- moved R25 15.6 mm to (51.3, 46.3), turned to 270 degrees
- moved C18 10.0 mm to (81.6, 43.5), turned to 270 degrees
- moved C1 6.03 mm to (23.9, 98.4)
- moved R3 5.62 mm to (56.2, 41.4), turned to 0 degrees
- moved J2 3.68 mm to (20.9, 76.8)
- moved R9 2.70 mm to (27.6, 49.6)
- moved C11 2.44 mm to (23.9, 111.5)
- moved R17 2.42 mm to (27.7, 45.6)
- moved D4 1.41 mm to (78.4, 55.8)
- moved R11 1.02 mm to (57.5, 47.6)
- moved R21 0.97 mm to (70.9, 42.9)
Connections:
- net Net-(D7-Pad2) renamed Csense
- C1 pad 1: Net-(C1-Pad1) -> Vout
- C11 pad 1: Net-(C1-Pad1) -> Vout
- C12 pad 1: Net-(C1-Pad1) -> Vout
- C18 pad 1: Net-(C18-Pad1) -> GND
- C18 pad 2: Net-(C18-Pad2) -> 15V
- C9 pad 1: Net-(C1-Pad1) -> Vout
- D10 pad 2: Net-(C18-Pad1) -> Net-(D10-Pad2)
- D11 pad 2: Net-(C18-Pad1) -> Net-(D10-Pad2)
- D3 pad 1: Net-(C1-Pad1) -> Vout
- J2 pad 1: Net-(C1-Pad1) -> Net-(D6-Pad1)
- L1 pad 2: Net-(C1-Pad1) -> Vout
- R21 pad 1: Net-(C18-Pad1) -> Net-(D10-Pad2)
- R25 pad 1: GND -> Vout
- R25 pad 2: Net-(C18-Pad2) -> Net-(C20-Pad2)
- R3 pad 1: Net-(C1-Pad1) -> Vout
- U3 pad 6: Net-(C18-Pad1) -> Net-(D10-Pad2)
Routing:
- net Vout: track 0.00 -> 95.9 mm, vias 0 -> 7
- net Net-(C1-Pad1): track 77.8 -> 0.00 mm, vias 7 -> 0
- net Net-(C18-Pad1): track 76.7 -> 0.00 mm, vias 3 -> 0
- net Net-(D10-Pad2): track 0.00 -> 75.5 mm, vias 0 -> 3
- net GND: track 75.3 -> 63.2 mm, vias 30 -> 29
- net CurrLimGND: track 15.2 -> 23.0 mm
- net Net-(C19-Pad1): track 13.8 -> 18.4 mm, vias 1 -> 2
- net Net-(R26-Pad2): track 8.41 -> 12.6 mm
- net Net-(--2-Pad1): track 41.1 -> 36.9 mm
- net Net-(C22-Pad1): track 19.4 -> 22.7 mm
- net Csense: track 37.5 -> 40.5 mm, vias 2 -> 3
- net 15V: track 173.1 -> 176.0 mm
- net Net-(C18-Pad2): track 2.49 -> 0.00 mm
- net Net-(C20-Pad2): track 0.00 -> 2.42 mm
- net FB: track 21.2 -> 22.9 mm, vias 0 -> 1
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- added copper zone on B.Cu, net Net-(D6-Pad1)
- added copper zone on F.Cu, net Net-(D6-Pad1)
- added copper zone on B.Cu, net Vout
- added copper zone on F.Cu, net Vout
- removed copper zone on B.Cu, net Net-(C1-Pad1)
- removed copper zone on F.Cu, net Net-(C1-Pad1)

Commit message: V3
Parts:
- removed C21: 470n, Capacitor_SMD:C_1206_3216Metric_Pad1.33x1.80mm_HandSolder
- removed D9: 100v, Diode_SMD:D_SMC_Handsoldering
- removed the R3 at (56.2, 41.4)
- removed the REF** at (76.7, 110.0)
- added D12: SMBJ100A, Diode_SMD:D_SMB, B.Cu at (80.1, 92.2)
- added R27: 0.2 5W, Resistor_THT:R_Radial_Power_L16.1mm_W9.0mm_P7.37mm, F.Cu at (24.3, 61.1)
- added R28: 1k, Resistor_SMD:R_1206_3216Metric_Pad1.30x1.75mm_HandSolder, B.Cu at (71.3, 40.6)
- added REF**: MountingHole_2.1mm, MountingHole:MountingHole_2.1mm, F.Cu at (21.6, 34.8)
- added REF**: MountingHole_2.1mm, MountingHole:MountingHole_2.1mm, F.Cu at (87.1, 117.6)
- added REF**: MountingHole_2.1mm, MountingHole:MountingHole_2.1mm, F.Cu at (20.8, 117.6)
- added REF**: MountingHole_2.1mm, MountingHole:MountingHole_2.1mm, F.Cu at (87.1, 35.1)
- added Rcl3: 1k, Resistor_SMD:R_0805_2012Metric, F.Cu at (32.8, 43.8)
- --1: value R -> inf
- --2: value R -> 0
- C13: value 100n -> 10u; footprint Capacitor_THT:CP_Radial_D18.0mm_P7.50mm -> Capacitor_THT:CP_Radial_D16.0mm_P7.50mm; moved to F.Cu
- C14: value 100n -> 10u; moved to F.Cu
- C9: renamed from C20; value C -> 1094pF
- D6: value 100v -> Dout; footprint Diode_SMD:D_SMC_Handsoldering -> Package_TO_SOT_THT:TO-220-3_Vertical
- L1: value 100uH -> 45uH
- R11: value 4.7k -> 3.3k
- R2: value 20k -> 50k
- R3: renamed from R1; value R -> 150k
- R6: value 10k -> 18k
- R7: value 22k -> 18k
- R9: renamed from R25; value 47k -> 1.73k
- moved C13 17.0 mm to (84.3, 108.7), turned to 180 degrees
- moved C14 7.40 mm to (84.3, 92.0), turned to 180 degrees
- moved R2 5.08 mm to (61.7, 41.7), turned to 90 degrees
- moved D7 1.85 mm to (32.8, 48.3)
- moved L1 1.67 mm to (61.5, 84.1)
- moved D6 1.26 mm to (27.5, 83.1), turned to -90 degrees
- renumbered C9 to C9in1, R9 to R9cl1
Connections:
- C13 pad 1: Vin -> GND
- C13 pad 2: GND -> Vin
- C14 pad 1: Vin -> GND
- C14 pad 2: GND -> Vin
- D3 pad 2: Net-(D3-Pad2) -> GND
- D6 pad 1: Net-(D6-Pad1) -> Vout
- D6 pad 2: Vout -> Net-(J2-Pad1)
- D7 pad 1: FB -> Net-(D7-Pad1)
- J2 pad 1: Net-(D6-Pad1) -> Net-(J2-Pad1)
- R14 pad 1: GND -> Vout
- R14 pad 2: Net-(D3-Pad2) -> GND
- R2 pad 1: GND -> Vout
- R2 pad 3: Net-(R2-Pad3) -> GND
- R21 pad 1: Net-(D10-Pad2) -> Net-(R21-Pad1)
- U2 pad 1: Net-(U2-Pad1) -> unconnected-(U2-Pad1)
- U2 pad 8: Net-(U2-Pad8) -> unconnected-(U2-Pad8)
- U3 pad 1: Net-(U3-Pad1) -> unconnected-(U3-Pad1)
- U3 pad 6: Net-(D10-Pad2) -> Net-(R21-Pad1)
- U3 pad 8: Net-(U3-Pad8) -> unconnected-(U3-Pad8)
Routing:
- net Net-(D10-Pad2): track 75.5 -> 56.7 mm, vias 3 -> 2
- net Net-(R21-Pad1): track 0.00 -> 14.7 mm, vias 0 -> 1
- net Vout: track 95.9 -> 101.4 mm
- net Net-(--2-Pad1): track 36.9 -> 32.9 mm, vias 1 -> 2
- net Net-(D3-Pad2): track 2.05 -> 0.00 mm
- net GND: track 63.2 -> 65.1 mm, vias 29 -> 28
- net Net-(D7-Pad1): track 0.00 -> 1.83 mm
- net FB: track 22.9 -> 24.1 mm
- net Csense: track 40.5 -> 41.1 mm
- net 15V: track 176.0 -> 175.3 mm
- net Vin: vias 8 -> 64
- net Net-(J2-Pad1): vias 0 -> 4
- net Net-(D6-Pad1): vias 4 -> 0
- net Net-(C4-Pad1): vias 0 -> 56
- added copper zone on B.Cu, net Net-(C4-Pad1)
- added copper zone on B.Cu, net Net-(J2-Pad1)
- added copper zone on F.Cu, net Net-(J2-Pad1)
- removed copper zone on B.Cu, net Net-(D6-Pad1)
- removed copper zone on F.Cu, net Net-(D6-Pad1)
Other:
- board outline added: 74.2 x 87.1 mm
- net class Default removed
